Commit message: Add files via upload

File: maker_robot/urdf/my_robot_car_4.xacro (robot description, xacro)
@@ -1,4 +1,4 @@
 <?xml version="1.0" ?>
-<robot name="my" xmlns:xacro="http://www.ros.org/wiki/xacro">
+<robot name="mobile_robot" xmlns:xacro="http://www.ros.org/wiki/xacro">
 <xacro:include filename="$(find maker_robot)/urdf/materials.xacro" />
 <material name="blue">
@@ -22,9 +22,4 @@
 </joint>
 <link name="base_plate">
-  <inertial>
-    <origin rpy="0 0 0" xyz="2.1363301386939105e-17 -0.0024965409300267195 0.04577001177847953"/>
-    <mass value="106.94277300466135"/>
-    <inertia ixx="1.844046" ixy="0.0" ixz="0.0" iyy="1.101918" iyz="1.3e-05" izz="2.804544"/>
-  </inertial>
   <visual>
     <origin rpy="0 0 0" xyz="0 0 0"/>
@@ -42,9 +37,4 @@
 </link>
 <link name="right_rear_wheel">
-  <inertial>
-    <origin rpy="0 0 0" xyz="0.0438314649294316 -2.4702462297909733e-15 1.734723475976807e-17"/>
-    <mass value="10.057534967035263"/>
-    <inertia ixx="0.046774" ixy="-0.0" ixz="-0.0" iyy="0.025998" iyz="0.0" izz="0.025998"/>
-  </inertial>
   <visual>
     <origin rpy="0 0 0" xyz="-0.175 0.17 -0.01"/>
@@ -62,9 +52,4 @@
 </link>
 <link name="right_front_wheel">
-  <inertial>
-    <origin rpy="0 0 0" xyz="0.04383146492943166 -2.55351295663786e-15 6.418476861114186e-17"/>
-    <mass value="10.05753496703526"/>
-    <inertia ixx="0.046774" ixy="-0.0" ixz="0.0" iyy="0.025998" iyz="0.0" izz="0.025998"/>
-  </inertial>
   <visual>
     <origin rpy="0 0 0" xyz="-0.175 -0.18 -0.01"/>
@@ -82,9 +67,4 @@
 </link>
 <link name="left_rear_wheel">
-  <inertial>
-    <origin rpy="0 0 0" xyz="-0.04383146492943163 -1.6681100944992977e-14 6.938893903907228e-17"/>
-    <mass value="10.057534967035268"/>
-    <inertia ixx="0.046774" ixy="0.0" ixz="-0.0" iyy="0.025998" iyz="-0.0" izz="0.025998"/>
-  </inertial>
   <visual>
     <origin rpy="0 0 0" xyz="0.175 0.17 -0.01"/>
@@ -102,9 +82,4 @@
 </link>
 <link name="left_front_wheel">
-  <inertial>
-    <origin rpy="0 0 0" xyz="-0.04383146492943174 -1.6653345369377348e-14 -1.9081958235744878e-17"/>
-    <mass value="10.057534967035286"/>
-    <inertia ixx="0.046774" ixy="0.0" ixz="-0.0" iyy="0.025998" iyz="-0.0" izz="0.025998"/>
-  </inertial>
   <visual>
     <origin rpy="0 0 0" xyz="0.175 -0.18 -0.01"/>
@@ -125,5 +100,5 @@
   <parent link="base_plate"/>
   <child link="right_front_wheel"/>
-  <axis xyz="-1.0 0.0 0.0"/>
+  <axis xyz="1.0 0.0 0.0"/>
 </joint>
 <joint name="right_front_wheel_joint" type="continuous">
@@ -131,5 +106,5 @@
   <parent link="base_plate"/>
   <child link="right_rear_wheel"/>
-  <axis xyz="-1.0 0.0 0.0"/>
+  <axis xyz="1.0 0.0 0.0"/>
 </joint>
 <joint name="left_rear_wheel_joint" type="continuous">
@@ -137,5 +112,5 @@
   <parent link="base_plate"/>
   <child link="left_front_wheel"/>
-  <axis xyz="-1.0 0.0 0.0"/>
+  <axis xyz="1.0 0.0 0.0"/>
 </joint>
 <joint name="left_front_wheel_joint" type="continuous">
@@ -143,5 +118,5 @@
   <parent link="base_plate"/>
   <child link="left_rear_wheel"/>
-  <axis xyz="-1.0 0.0 0.0"/>
+  <axis xyz="1.0 0.0 0.0"/>
 </joint>
 <joint name="laser_joint" type="fixed">
